File: hw/PGA.kicad_sch (KiCad schematic)
At the start: 11 parts, among them U301 MAX9939AUB+T

Commit message: Starting some layout
Parts:
- U301: footprint symbols:21-0061L_MXM -> Library:SOP50P490X110-10N
- renumbered C312 to C302, C314 to C303, C315 to C304, C316 to C305, C317 to C306, R309 to R304
Changed lines of the file:
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@@
 		(on_board yes)
 		(dnp no)
-		(property "Reference" "R309"
+		(property "Reference" "R304"
 			(at 176.53 99.314 90)
 			(effects
@@
 			(project "NexVLF"
 				(path "/c3add214-400b-4323-a350-6b93b7811d69/056d8594-8686-488d-8212-c8ea658b316d"
-					(reference "R309")
+					(reference "R304")
 					(unit 1)
 				)
@@
 		(on_board yes)
 		(dnp no)
-		(property "Reference" "C312"
+		(property "Reference" "C302"
 			(at 159.258 73.914 0)
 			(effects
@@
 			(project "NexVLF"
 				(path "/c3add214-400b-4323-a350-6b93b7811d69/056d8594-8686-488d-8212-c8ea658b316d"
-					(reference "C312")
+					(reference "C302")
 					(unit 1)
 				)
@@
 		(on_board yes)
 		(dnp no)
-		(property "Reference" "C314"
+		(property "Reference" "C303"
 			(at 159.258 90.424 0)
 			(effects
@@
 			(project "NexVLF"
 				(path "/c3add214-400b-4323-a350-6b93b7811d69/056d8594-8686-488d-8212-c8ea658b316d"
-					(reference "C314")
+					(reference "C303")
 					(unit 1)
 				)
@@
 		(on_board yes)
 		(dnp no)
-		(property "Reference" "C317"
+		(property "Reference" "C306"
 			(at 180.594 104.394 0)
 			(effects
@@
 			(project "NexVLF"
 				(path "/c3add214-400b-4323-a350-6b93b7811d69/056d8594-8686-488d-8212-c8ea658b316d"
-					(reference "C317")
+					(reference "C306")
 					(unit 1)
 				)
@@
 		(on_board yes)
 		(dnp no)
-		(property "Reference" "C316"
+		(property "Reference" "C305"
 			(at 98.044 96.774 0)
 			(effects
@@
 			(project "NexVLF"
 				(path "/c3add214-400b-4323-a350-6b93b7811d69/056d8594-8686-488d-8212-c8ea658b316d"
-					(reference "C316")
+					(reference "C305")
 					(unit 1)
 				)
@@
 		(on_board yes)
 		(dnp no)
-		(property "Reference" "C315"
+		(property "Reference" "C304"
 			(at 92.71 96.774 0)
 			(effects
@@
 			(project "NexVLF"
 				(path "/c3add214-400b-4323-a350-6b93b7811d69/056d8594-8686-488d-8212-c8ea658b316d"
-					(reference "C315")
+					(reference "C304")
 					(unit 1)
 				)
@@
 			)
 		)
-		(property "Footprint" "symbols:21-0061L_MXM"
+		(property "Footprint" "Library:SOP50P490X110-10N"
 			(at 106.68 68.58 0)
 			(effects
