File: hw/NexVLF.kicad_pcb (KiCad board)
At the start: 6 copper layers, 96 x 61 mm, 148 parts, among them J501 68710814022, J502 FTSH-105-01-L-DV-K, J601 pwr+data, Q101 2N7002, Q102 2N7002, Q103 2N7002, Q104 2N7002, Q105 2N7002, SW501 Push button switch, U101 AK5572EN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

Commit message: Routing complete for DVT1 all ERC and DRC pass, 3D view is full
Parts:
- removed C114: 1uF, Capacitor_SMD:C_0402_1005Metric
- removed C115: 100nF, Capacitor_SMD:C_0402_1005Metric
- removed Q105: 2N7002, Package_TO_SOT_SMD:SOT-23
- added D102: 1SV149, Package_TO_SOT_THT:TO-92-2, F.Cu at (97.9, 86.5)
- added J101: ANT, TerminalBlock_Altech:Altech_AK300_1x02_P5.00mm_45-Degree, F.Cu at (100.0, 91.9)
- added Q106: DMN32D2LDF, Package_TO_SOT_SMD:SOT-353_SC-70-5, F.Cu at (111.5, 67.0)
- added R107: 22, Resistor_SMD:R_0402_1005Metric, F.Cu at (124.9, 73.5)
- added R108: 1M, Resistor_SMD:R_0402_1005Metric, F.Cu at (113.8, 66.8)
- added R109: 1M, Resistor_SMD:R_0402_1005Metric, F.Cu at (109.4, 78.0)
- added R110: 1M, Resistor_SMD:R_0402_1005Metric, F.Cu at (109.4, 81.4)
- added R111: 1M, Resistor_SMD:R_0402_1005Metric, F.Cu at (111.9, 75.1)
- added R112: 1M, Resistor_SMD:R_0402_1005Metric, F.Cu at (109.4, 85.9)
- added R526: 100k, Resistor_SMD:R_0402_1005Metric, F.Cu at (134.5, 109.6)
- added R527: 100, Resistor_SMD:R_0402_1005Metric, F.Cu at (134.1, 111.3)
- C112: value 1uF -> 10uF
- Q101, Q102, Q103, Q104: value 2N7002 -> DMN32D2LDF; footprint Package_TO_SOT_SMD:SOT-23 -> Package_TO_SOT_SMD:SOT-353_SC-70-5
- R520, R605, R606, R607, R608: footprint Resistor_SMD:R_0603_1608Metric -> Resistor_SMD:R_0402_1005Metric
- moved R520 259.6 mm to (170.1, 104.9), turned to 90 degrees
- moved C506 257.4 mm to (172.3, 108.2)
- moved C507 257.3 mm to (172.3, 109.2), turned to 180 degrees
- moved C510 253.8 mm to (171.6, 105.8), turned to -90 degrees
- moved C508 250.7 mm to (166.1, 105.0)
- moved C513 250.4 mm to (169.0, 100.1)
- moved C511 250.3 mm to (167.7, 111.7), turned to -90 degrees
- moved C528 249.6 mm to (174.1, 89.2), turned to 90 degrees
- moved C509 248.0 mm to (165.7, 104.0), turned to 180 degrees
- moved C512 247.4 mm to (165.7, 102.1), turned to 180 degrees
- moved C515 245.4 mm to (155.5, 99.1)
- moved C514 243.6 mm to (150.3, 115.4), turned to -90 degrees
- moved C517 240.7 mm to (151.5, 96.3), turned to 90 degrees
- moved R518 235.2 mm to (171.7, 102.6), turned to -90 degrees
- moved R521 233.6 mm to (172.3, 91.6)
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Connections:
- net /tuneVoltage renamed /Microcontroller/tuneVoltage
- C101 pad 2: /rf+ -> /PGA1/in+
- C104 pad 2: Net-(Q105-D) -> Net-(Q104-D1)
- C105 pad 2: Net-(Q102-D) -> Net-(Q101-D1)
- C106 pad 2: Net-(Q103-D) -> Net-(Q102-D1)
- C107 pad 2: Net-(Q103-D) -> Net-(Q102-D1)
- C108 pad 2: Net-(Q104-D) -> Net-(Q103-D1)
- C109 pad 2: Net-(Q104-D) -> Net-(Q103-D1)
- C110 pad 2: Net-(Q101-D) -> Net-(Q106-D1)
- C111 pad 2: Net-(Q104-D) -> Net-(Q103-D1)
- D101 pad 1: GND -> /varactorVoltage
- D101 pad 2: /rf+ -> GND
- Q101 pad 1: /Cbank0 -> /Cbank1
- Q101 pad 2: GND -> Net-(Q101-S)
- Q101 pad 3: Net-(Q101-D) -> /Cbank1
- Q102 pad 1: /Cbank1 -> /Cbank2
- Q102 pad 2: GND -> Net-(Q102-S)
- Q102 pad 3: Net-(Q102-D) -> /Cbank2
- Q103 pad 1: /Cbank2 -> /Cbank3
- Q103 pad 2: GND -> Net-(Q103-S)
- Q103 pad 3: Net-(Q103-D) -> /Cbank3
- Q104 pad 1: /Cbank3 -> /Cbank4
- Q104 pad 2: GND -> Net-(Q104-S)
- Q104 pad 3: Net-(Q104-D) -> /Cbank4
- SW501 pad 3: (no net) -> Net-(R521-Pad2)
- SW501 pad 4: (no net) -> /Microcontroller/BOOT0
- U301 pad 5: /rf+ -> /PGA1/in+
- U501 pad 22: unconnected-(U501-PA0-Pad22) -> Net-(U501-PA0)
Routing:
- net GND: track 0.00 -> 158.3 mm, vias 0 -> 117
- net /Microcontroller/dispNSS: track 0.00 -> 93.1 mm
- net /Microcontroller/dispSCK: track 0.00 -> 87.5 mm, vias 0 -> 2
- net /Microcontroller/SWCL: track 0.00 -> 84.8 mm, vias 0 -> 2
- net /Microcontroller/dispDC: track 0.00 -> 80.2 mm, vias 0 -> 2
- net /Microcontroller/dispRESET: track 0.00 -> 77.1 mm, vias 0 -> 2
- net /Microcontroller/SWDIO: track 0.00 -> 73.9 mm, vias 0 -> 2
- net /Cbank3: track 0.00 -> 67.5 mm, vias 0 -> 2
- net /Microcontroller/nBLU: track 0.00 -> 64.7 mm, vias 0 -> 2
- net /Cbank1: track 0.00 -> 62.4 mm, vias 0 -> 2
- net nRESET: track 0.00 -> 61.6 mm, vias 0 -> 4
- net /Cbank0: track 0.00 -> 61.1 mm, vias 0 -> 2
- net /Microcontroller/nRED: track 0.00 -> 59.3 mm, vias 0 -> 2
- net /Microcontroller/nGRN: track 0.00 -> 58.5 mm, vias 0 -> 2
- net /Cbank2: track 0.00 -> 58.5 mm, vias 0 -> 2
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- added copper zone on In3.Cu, net +3.3V
- added copper zone on In3.Cu, net +3.3VA
- added copper zone on In3.Cu, net +5VA
- added copper zone on In3.Cu, net /Power/+5.4V-dirty
- added copper zone on In1.Cu, net GND
- added copper zone on In4.Cu, net GND
- added copper zone on In3.Cu, net VBUS
Other:
- board text added: "1pF gimmick"
