File: hw/power.kicad_sch (KiCad schematic)
At the start: 35 parts, among them J1501 pwr+data, U1502 LMR51430, U1503 TPS22918DBVR, U1506 TPS61023, U1507 TPS7A2050PDBVR, U1508 TPS7A2033PDBVR

Commit message: Starting some layout
Parts:
- removed C1504: 1uF, Capacitor_SMD:C_0402_1005Metric, symbol Device:C
- removed C1508: 220pF, Capacitor_SMD:C_0603_1608Metric, symbol Device:C
- removed U1503: TPS22918DBVR, Library:SOT95P280X145-6N, symbol Library:TPS22918DBVR
- U603: renamed from U1507; symbol Library:PTPS7A2012PDBVR -> Library:PTPS7A20xxPDBVR
- U604: renamed from U1508; symbol Library:PTPS7A2012PDBVR -> Library:PTPS7A20xxPDBVR
- renumbered C1501 to C601, C1502 to C602, C1503 to C603, C1506 to C604, C1507 to C605, C1518 to C606, C1520 to C607, C1521 to C608, C1522 to C609, C1523 to C610, C1524 to C611, C1525 to C612, C1526 to C613, D1501 to D601, D1502 to D602, D1503 to D603, FB1501 to FB601, J1501 to J601, L1501 to L601, L1502 to L602, R1501 to R601, R1502 to R602, R1507 to R603, R1508 to R604, R1509 to R605, R1510 to R606, R1511 to R607, R1512 to R608, U1502 to U601, U1506 to U602
Connections:
- net +3.3V-ON is gone; now on net +3.3V: C604.1, C605.1, L601.2, R601.2
Other:
- note removed: "+3.3V load switch"
- note removed: "~455us 3.3V rise time"

Commit message: Routing complete for DVT1 all ERC and DRC pass, 3D view is full
Parts:
- R605, R606, R607, R608: footprint Resistor_SMD:R_0603_1608Metric -> Resistor_SMD:R_0402_1005Metric
Changed lines of the file:
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@@
 			)
 		)
-		(property "Footprint" "Resistor_SMD:R_0603_1608Metric"
+		(property "Footprint" "Resistor_SMD:R_0402_1005Metric"
 			(at 125.476 188.214 90)
 			(effects
@@
 			)
 		)
-		(property "Footprint" "Resistor_SMD:R_0603_1608Metric"
+		(property "Footprint" "Resistor_SMD:R_0402_1005Metric"
 			(at 134.366 175.514 90)
 			(effects
@@
 			)
 		)
-		(property "Footprint" "Resistor_SMD:R_0603_1608Metric"
+		(property "Footprint" "Resistor_SMD:R_0402_1005Metric"
 			(at 106.934 188.214 90)
 			(effects
@@
 			)
 		)
-		(property "Footprint" "Resistor_SMD:R_0603_1608Metric"
+		(property "Footprint" "Resistor_SMD:R_0402_1005Metric"
 			(at 106.934 175.514 90)
 			(effects
